Commit message: ok

File: moveit_arm_bot/catkin_ws/src/mon_robot_moveit/urdf/robot.urdf (robot description, URDF)
Before this commit: robot robot_4axes, 6 links, 5 joints
Links:
- added link link_5; visual box size=0.05 0.05 0.03
- added link link_6; visual cylinder length=0.03 radius=0.02
- link base_link: geometry visual cylinder length=0.05 radius=0.1
- link finger_l: geometry visual box size=0.01 0.02 0.04
- link link_1: geometry visual cylinder length=0.1 radius=0.05
- link link_2: geometry visual box size=0.04 0.04 0.3
- link link_3: geometry visual box size=0.03 0.03 0.2
- link link_4: geometry visual cylinder length=0.06 radius=0.025
Joints:
- removed joint gripper_joint
- added joint finger_joint: type prismatic, parent link_6, child finger_l, origin xyz=0 0 0.03 rpy=0 0 0, axis 1 0 0, limit lower=0.0 upper=0.05 effort=50.0 velocity=0.1
- added joint joint_5: type revolute, parent link_4, child link_5, origin xyz=0 0 0.06 rpy=0 0 0, axis 0 0 1, limit lower=-3.1416 upper=3.1416 effort=50.0 velocity=1.5
- added joint joint_6: type revolute, parent link_5, child link_6, origin xyz=0 0 0.03 rpy=0 0 0, axis 0 1 0, limit lower=-1.5708 upper=1.5708 effort=50.0 velocity=1.5
- joint elbow_joint: limit lower=-1.57 upper=1.57 effort=100 velocity=1.0 -> lower=-2.0944 upper=2.0944 effort=150.0 velocity=1.0; origin xyz=0 0 0.2 rpy=0 0 0 -> xyz=0 0 0.3 rpy=0 0 0
- joint shoulder_joint: limit lower=-1.57 upper=1.57 effort=100 velocity=1.0 -> lower=-1.5708 upper=1.5708 effort=150.0 velocity=1.0; origin xyz=0 0 0.2 rpy=0 0 0 -> xyz=0 0 0.1 rpy=0 0 0
- joint waist_joint: limit lower=-3.14 upper=3.14 effort=100 velocity=1.0 -> lower=-3.1416 upper=3.1416 effort=150.0 velocity=1.0; origin xyz=0 0 0.05 rpy=0 0 0 -> xyz=0 0 0.025 rpy=0 0 0
- joint wrist_joint: limit lower=-3.14 upper=3.14 effort=100 velocity=1.0 -> lower=-1.7453 upper=1.7453 effort=100.0 velocity=1.0
