Commit message: ok

File: moveit_arm_bot/catkin_ws/src/mon_robot_moveit/urdf/robot_visual.urdf (robot description, URDF)
Before this commit: robot robot_4axes, 1 links, 0 joints
Links:
- added link link_1; visual mesh filename=../meshes/ok.stl scale=0.001 0.001 0.001
- link base_link: geometry 
Joints:
- added joint waist_joint: type revolute, parent base_link, child link_1, origin xyz=0 0 0.025 rpy=0 0 0, axis 0 0 1, limit lower=-3.1416 upper=3.1416 effort=150.0 velocity=1.0
